Commit message: refactor: tidy file system, change the package name to lidar_diffbot_description, add placeholder lidar_diffbot_navigation package.

File: lidar_diffbot_description/urdf/colored_lidar_diffbot.urdf (robot description, URDF)
Before this commit: robot lidar_diffbot, 7 links, 6 joints
Links:
- link base_link: geometry collision mesh filename=package://lidar_diffbot_description/meshes/collision/base_l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; visual mesh filename=package://lidar_diffbot_description/meshes/visual/base_link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
- link caster_wheel_link: geometry collision mesh filename=package://lidar_diffbot_description/meshes/collision/caster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; visual mesh filename=package://lidar_diffbot_description/meshes/visual/caster_wh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
- link imu_link: geometry collision mesh filename=package://lidar_diffbot_description/meshes/collision/imu_li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; visual mesh filename=package://lidar_diffbot_description/meshes/visual/imu_link.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
- link laser_link: geometry collision mesh filename=package://lidar_diffbot_description/meshes/collision/laser_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; visual mesh filename=package://lidar_diffbot_description/meshes/visual/laser_lin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
- link left_wheel_link: geometry collision mesh filename=package://lidar_diffbot_description/meshes/collision/left_w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; visual mesh filename=package://lidar_diffbot_description/meshes/visual/left_whee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
- link right_wheel_link: geometry collision mesh filename=package://lidar_diffbot_description/meshes/collision/right_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; visual mesh filename=package://lidar_diffbot_description/meshes/visual/right_whe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

Commit message: fix(urdf): fix base_link_joint

File: lidar_diffbot_description/urdf/colored_lidar_diffbot.urdf (robot description, URDF)
Before this commit: robot lidar_diffbot, 7 links, 6 joints
Joints:
- joint base_footprint_joint: origin xyz=0.0 0.0 0.0 rpy=0.0 0.0 0.0 -> xyz=0.0 0.0 0.0325 rpy=0.0 0.0 0.0

File: lidar_diffbot_description/urdf/lidar_diffbot.urdf (robot description, URDF)
Before this commit: robot lidar_diffbot, 7 links, 6 joints
Joints:
- joint base_footprint_joint: origin xyz=0.0 0.0 0.0 rpy=0.0 0.0 0.0 -> xyz=0.0 0.0 0.0325 rpy=0.0 0.0 0.0

Commit message: refactor(desc): rename laser_link into laser_frame for ydlidar driver convention

File: lidar_diffbot_description/urdf/colored_lidar_diffbot.urdf (robot description, URDF)
Before this commit: robot lidar_diffbot, 7 links, 6 joints
Links:
- removed link laser_link
- added link laser_frame, mass 0.0; collision mesh filename=package://lidar_diffbot_description/meshes/collision/laser_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; visual mesh filename=package://lidar_diffbot_description/meshes/visual/laser_fra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
Joints:
- joint lidar_joint: child laser_link -> laser_frame

File: lidar_diffbot_description/urdf/lidar_diffbot.urdf (robot description, URDF)
Before this commit: robot lidar_diffbot, 7 links, 6 joints
Links:
- removed link laser_link
- added link laser_frame, mass 0.0; collision mesh filename=package://lidar_diffbot_description/meshes/collision/laser_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; visual mesh filename=package://lidar_diffbot_description/meshes/collision/laser_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
Joints:
- joint lidar_joint: child laser_link -> laser_frame
